Commit message: Save complete new project version

File: uam_ocp/models/generated/uam_pinocchio.urdf (robot description, URDF)
Before this commit: robot iris, 20 links, 19 joints
Joints:
- joint shoulder_pan_joint: axis 0 0 1 -> (none); limit lower=-1.57 upper=1.57 effort=1000 velocity=2 -> (none); type revolute -> fixed
